File: control-matrix/control-matrix-2.kicad_pcb (KiCad board)
At the start: 2 copper layers, 60 x 30 mm, 9 parts, among them J1 Screw_Terminal_01x02, J2 Screw_Terminal_01x02, J9 Screw_Terminal_01x02, SW1 SW_Rotary_1x12

Commit message: control-matrix: add power input labels on silkscreen
Other:
- board text added: "GND +12V"
Changed lines of the file:
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@@
 		(layer "Edge.Cuts")
+	)
+	(gr_text "GND  +12V"
+		(at 110.4 81.6 0)
+		(layer "F.SilkS")
+		(effects
+			(font
+				(size 1 1)
+				(thickness 0.2)
+				(bold yes)
+			)
+			(justify left bottom)
+		)
 	)
 	(segment

Commit message: control-matrix: add ground planes
This avoids having to etch too much copper.
Routing:
- net GND: track 27.9 -> 0.00 mm
- added copper zone on F.Cu, net GND
Changed lines of the file:
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@@
-	)
-	(segment
-		(start 112.06 92.94)
-		(end 110.2 94.8)
-		(width 0.4)
-		(layer "F.Cu")
-		(net 11)
-	)
-	(segment
-		(start 112.06 84.1)
-		(end 112.06 92.94)
-		(width 0.4)
-		(layer "F.Cu")
-		(net 11)
-	)
-	(segment
-		(start 110.2 94.8)
-		(end 97.70533 94.8)
-		(width 0.4)
-		(layer "F.Cu")
-		(net 11)
-	)
-	(segment
-		(start 97.70533 94.8)
-		(end 94.90475 97.60058)
-		(width 0.4)
-		(layer "F.Cu")
-		(net 11)
 	)
 	(segment
@@
 		(net 12)
 	)
+	(zone
+		(net 11)
+		(net_name "GND")
+		(layer "F.Cu")
+		(hatch edge 0.5)
+		(connect_pads
+			(clearance 0.5)
+		)
+		(min_thickness 0.25)
+		(filled_areas_thickness no)
+		(fill yes
+			(thermal_gap 0.5)
+			(thermal_bridge_width 0.5)
+		)
+		(polygon
+			(pts
+				(xy 58.4 78.2) (xy 123.3 78.4) (xy 123.3 112) (xy 58.4 111.3)
+			)
+		)
+	)
 	(embedded_fonts no)
