File: control-matrix/control-matrix-4.kicad_pcb (KiCad board)
At the start: 2 copper layers, 90 x 30 mm, 16 parts, among them J1 Screw_Terminal_01x02, J2 Screw_Terminal_01x02, J3 Screw_Terminal_01x02, J4 Screw_Terminal_01x02, J9 Screw_Terminal_01x02, SW1 SW_Rotary_1x12

Commit message: control-matrix: add power input labels on silkscreen
Other:
- board text added: "GND +12V"
Changed lines of the file:
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@@
 		(layer "Edge.Cuts")
+	)
+	(gr_text "GND  +12V"
+		(at 140.4 81.6 0)
+		(layer "F.SilkS")
+		(effects
+			(font
+				(size 1 1)
+				(thickness 0.2)
+				(bold yes)
+			)
+			(justify left bottom)
+		)
 	)
 	(segment

Commit message: control-matrix: add ground planes
This avoids having to etch too much copper.
Routing:
- net GND: track 27.9 -> 0.00 mm
- added copper zone on B.Cu, net GND
- added copper zone on F.Cu, net GND
Changed lines of the file:
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@@
-	)
-	(segment
-		(start 142.06 92.94)
-		(end 140.2 94.8)
-		(width 0.4)
-		(layer "F.Cu")
-		(net 13)
-	)
-	(segment
-		(start 142.06 84.1)
-		(end 142.06 92.94)
-		(width 0.4)
-		(layer "F.Cu")
-		(net 13)
-	)
-	(segment
-		(start 140.2 94.8)
-		(end 127.70533 94.8)
-		(width 0.4)
-		(layer "F.Cu")
-		(net 13)
-	)
-	(segment
-		(start 127.70533 94.8)
-		(end 124.90475 97.60058)
-		(width 0.4)
-		(layer "F.Cu")
-		(net 13)
 	)
 	(segment
@@
 		(net 14)
 	)
+	(zone
+		(net 13)
+		(net_name "GND")
+		(layers "F.Cu" "B.Cu")
+		(hatch edge 0.5)
+		(connect_pads
+			(clearance 0.5)
+		)
+		(min_thickness 0.25)
+		(filled_areas_thickness no)
+		(fill yes
+			(thermal_gap 0.5)
+			(thermal_bridge_width 0.5)
+		)
+		(polygon
+			(pts
+				(xy 59.1 79.2) (xy 151.2 78.8) (xy 151.3 110.9) (xy 58.8 110.7)
+			)
+		)
+	)
 	(group ""
